File: NetworkNotifier/NetworkNotifier.kicad_pcb (KiCad board)
At the start: 2 copper layers, 55 x 25 mm, 50 parts, among them J1 Conn_01x06, J2 USB_B_Micro, J3 RJ45_Hanrun_HR911105A_Horizon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, J4 Conn_01x04, SW1 SW_Push, U1 W5500, U2 STM32G031K8Tx, U3 SN74LVC2G14DBV, U4 SN74LVC2G14DBV, U6 AP2112K-3.3, Y1 25 MHz

Commit message: Very rough placing done
Parts:
- J1: footprint Connector_PinHeader_2.54mm:PinHeader_1x05_P2.54mm_Vertical -> Connector_PinHeader_2.54mm:PinHeader_1x06_P2.54mm_Vertical
- moved C8 35.7 mm to (132.3, 79.2)
- moved D1 33.9 mm to (112.1, 88.8), turned to 0 degrees
- moved C7 33.7 mm to (140.6, 70.8), turned to 180 degrees
- moved C11 33.4 mm to (135.7, 79.0)
- moved R5 33.4 mm to (113.2, 86.5), turned to 180 degrees
- moved D2 32.8 mm to (116.2, 87.9)
- moved D6 31.0 mm to (112.2, 84.5), turned to 0 degrees
- moved D3 31.0 mm to (120.8, 87.9)
- moved R6 30.9 mm to (118.5, 87.6), turned to -90 degrees
- moved D4 29.8 mm to (125.2, 87.9)
- moved R10 29.3 mm to (115.8, 84.5)
- moved R7 29.3 mm to (123.0, 87.6), turned to -90 degrees
- moved R8 27.7 mm to (127.5, 87.6)
- moved C12 26.7 mm to (140.5, 87.5), turned to 90 degrees
- moved C2 26.0 mm to (147.8, 85.0)
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